File: Hardware Files/MicroBBPS.kicad_pcb (KiCad board)
At the start: 2 copper layers, 54 x 24 mm, 23 parts, among them J2 USB_B_Micro, J3 Conn_02x03, J4 Conn_02x03, J5 Conn_01x02, J8 3PoleHeaderSwitch, J9 3PoleHeaderSwitch, U1 NCP1117ST50T3G, U3 NCP1117ST33T3G

Commit message: Adding USB-C Files
Parts:
- removed J2: USB_B_Micro, MicroBBPS:U-F-M5DD-Y-L
- added J1: USB_C_Receptacle_PowerOnly_6P, Library:GT-USB-7002C, F.Cu at (21.5, 6.60)
- added R3: 5k 0.25W, Resistor_SMD:R_0402_1005Metric, F.Cu at (19.5, 9.10)
- added R4: 5k 0.25W, Resistor_SMD:R_0402_1005Metric, F.Cu at (23.5, 9.10)
- D1, D3: value LED -> Green 3.0V
- D2: value D -> 400V 1A SMA
- J5: value Conn_01x02 -> Screw Terminal
- R1: value 56R 0.25W -> 10k 0.25W
- R2: value 0R -> 10k 0.25W
- moved J3 0.25 mm to (3.12, 20.0)
Connections:
- net +3V3 renamed +3.3V
- net /VoutLeft renamed VoutLeft
- net /VoutRight renamed VoutRight
Routing:
- net +3.3V: track 49.1 -> 67.8 mm, vias 1 -> 2
- net +5V: track 70.2 -> 86.7 mm
- net /CC2: track 0.00 -> 3.41 mm
- net /CC1: track 0.00 -> 3.41 mm
Other:
- outline, holes or cut-outs redrawn
- net class Default removed
